File: Eagle/self leveling tray schematic.brd (EAGLE design)
At the start: 100 x 80 mm, 9 parts

Commit message: Schematic Version 1.2
Added changes suggested by Andrew.
Added LEDs and grounded unused GPIO.

Email from Andrew:
Hi Taylor!

> Could you take a look at our current schematic? It passes ERC right
now,
> but I'm not sure if I'm missing something critical.

- You need 100 nF bypass caps on the 328's VCC and AVCC pins.
- Use a 3.3V supply symbol, not wires, for your supply.
- Your regulator absolutely needs filter caps - large filter caps. Read
the data sheet.
- What's your battery voltage? what kind of batteries? note it in the
schematic.
- What kind of accelerometer? Note it in the schermatic.
- No crystal, so you're using the internal RC oscilator
Parts:
- added BYPASS_CAP_1, BYPASS_CAP_2: 100 nF, rcl:C1206
- added LED1_GREEN, LED2_YELLOW, LED3_YELLOW, LED4_RED: TBD Voltage, led:1206
- added LED_RESISTOR_1, LED_RESISTOR_2, LED_RESISTOR_3, LED_RESISTOR_4: TBD Resistance, rcl:R1206
- renumbered PIN_ACCELEROMETER to PIN_ACCELEROMETER_MMA8452Q, PIN_SERVO to PIN_SERV_CTRL_MICRO_MAESTRO, PIN_VCC_REGULATOR to PIN_VCC_REGULATOR_D24V5F3
Connections:
- net BATTERY_VCC renamed 6V_BATTERY_VCC
- removed net 3.3V_VCC: ATMEGA328.20, ATMEGA328.7, DRAGON_ISP.5, PIN_ACCELEROMETER_MMA8452Q.1, PIN_VCC_REGULATOR_D24V5F3.4, PULL_UP_2.2
- new net LED_OUT_1: ATMEGA328.13, LED_RESISTOR_1.1
- new net LED_OUT_2: ATMEGA328.12, LED_RESISTOR_2.1
- new net LED_OUT_3: ATMEGA328.11, LED_RESISTOR_3.1
- new net LED_OUT_4: ATMEGA328.6, LED_RESISTOR_4.1
- new net N$2: LED1_GREEN.A, LED_RESISTOR_1.2
- new net N$3: LED2_YELLOW.A, LED_RESISTOR_2.2
- new net N$4: LED3_YELLOW.A, LED_RESISTOR_3.2
- new net N$5: LED4_RED.A, LED_RESISTOR_4.2
- new net VCC: ATMEGA328.20, ATMEGA328.7, BYPASS_CAP_1.1, BYPASS_CAP_2.1, DRAGON_ISP.5, PIN_ACCELEROMETER_MMA8452Q.1, PIN_VCC_REGULATOR_D24V5F3.4, PULL_UP_2.2
- net GND: now also ATMEGA328.14, ATMEGA328.15, ATMEGA328.16, ATMEGA328.23, ATMEGA328.24, ATMEGA328.25, ATMEGA328.26, BYPASS_CAP_1.2, BYPASS_CAP_2.2, LED1_GREEN.C, LED2_YELLOW.C, LED3_YELLOW.C, LED4_RED.C
Routing:
- net 3.3V_VCC: track 95.5 -> 0.00 mm
